File: Heater-Control/boards/controller/Heater_Control_v2.brd (EAGLE design)
At the start: 40.6 x 36.8 mm, 4 parts, among them J1 S2B-XH-A(LF)(SN), U1 QT Py #4600, X1 MLX-43860

Commit message: updated control board
Parts:
- removed X1: MLX-43860, home:MLX-43860
- added J2: S2B-XH-A(LF)(SN), Connectors:HDR-02/RA
- added Q1: TP2104N3-G, home:TO92-
- added R2: 100, home:R1206
- J1: value S2B-XH-A(LF)(SN) -> MLX-43860; device Connectors:HDR-02/RA -> home:MLX-43860
- R1: value 4.7k -> 3.3k
- moved J1 15.5 mm to (6.35, 12.7)
Connections:
- new net GATE: Q1.2, R2.2
- new net SPU_GATE: R2.1, U1.A2@1, U1.A2@2
- net 3V3: now also Q1.1
- net DATA-1WIRE: now also J1.2, J1.3, Q1.3; no longer X1.2, X1.3
- net GND: now also J1.1, J1.4, J2.2; no longer J1.2, X1.1, X1.4
- net PWR: now also J2.1; no longer J1.1
Routing:
- net 3V3: track 17.1 -> 37.4 mm
- net DATA-1WIRE: track 42.1 -> 51.1 mm
- net GATE: track 0.00 -> 8.23 mm
- net SPU_GATE: track 0.00 -> 6.50 mm
- net PWR: track 32.6 -> 33.1 mm
Other:
- board text added: "1-Wire Heater Control"
- board text added: "1-wire sensors"
- board text added: "Rev 2b"
- board text added: "power strip"
- board text added: "strong pull-up"
